File: Precharge/precharge.kicad_sch (KiCad schematic)
At the start: 31 parts, among them J1 AIR_CONN, J2 TSAL_CONN_AIR, J3 TSAL_CONN_LV, J4 LV_CONN, J5 HV_CONN, J6 CAP_CONN, K1 IMB06IGR, Q1 AM2328NE, Q2 SQ2362, Q3 SQ2362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

Commit message: Add files via upload
Parts:
- removed K1: IMB06IGR, customFootprints:IMB03IGR, symbol Relay:Relay_SPST-NO
- removed Q1: AM2328NE, customFootprints:SOT95P237X112-3N, symbol Device:Q_NMOS_GSD
- removed Q2, Q3: SQ2362, customFootprints:SOT95P237X112-3N, symbol Device:Q_NMOS_GSD
- removed R19, R20, R22: 1K, Resistor_SMD:R_0805_2012Metric, symbol Device:R_Small
- removed R21: 15K, customFootprints:PWR263S-35-1002F_BRN, symbol Device:Heater
- removed RN10K1: 10K, customFootprints:GULLWING24_VIS, symbol customSymbols:OSOPTC1002AT0
- removed U3: MC34074ADR2G, customFootprints:SOIC127P600X175-14N, symbol Device:Opamp_Quad
- added D1, D4: 1N4448X-TP, Diode_SMD:D_SOD-523, symbol Device:D_Small
- added D2: 151031VS06000, customFootprints:WL-TMRC_3MM, symbol Device:LED_Small
- added D3: 151031SS06000, customFootprints:WL-TMRC_3MM, symbol Device:LED_Small
- added K1: 12V, customFootprints:RELAY_G9KB-1A_OMR, symbol customSymbols:G9KB-1A_DC12
- added Q1: SI1539CDL-T1-GE3, Package_SO:SOIC-8_3.9x4.9mm_P1.27mm, symbol Transistor_FET:Si4542DY
- added R10, R11, R12, R13, R14, R15, R9: 10K, Resistor_SMD:R_0805_2012Metric, symbol Device:R_Small
- added R16, R17: 600, Resistor_SMD:R_0805_2012Metric, symbol Device:R_Small
- added R7: 15K, customFootprints:PWR263S-35-1002F_BRN, symbol Device:Heater
- added U3: MC33072DR2G, customFootprints:SOIC127P600X175-8N, symbol Device:Opamp_Dual
- added U4: TL331, Package_TO_SOT_SMD:SOT-23-5, symbol Comparator:TL331
- J1: value AIR_CONN -> CONN_AIR
- J4: value LV_CONN -> CONN_LV
- J5: value HV_CONN -> CONN_HV
- J6: value CAP_CONN -> CONN_CAP
- R1, R4: value 187K -> 124K; Model CRCW2512187KFKEG -> CRCW2512124KFKEG
- R2, R5: value 11K -> 110K; Model CRCW251211K0FKEG -> CRCW2512110KFKEG
- renumbered R14 to R8
Connections:
- net +12V: now also Q1.4 (1), U3.8 (V+), U4.5 (V+)
- net AIR+: now also D2.2 (A), D4.1 (K), Q1.2 (G), Q1.5 (G), U4.4
- net LVGND: now also D1.2 (A), D4.2 (A), K1.1, Q1.1 (S), R11.1, R15.1, R16.2, R17.2, U3.4 (V-), U4.2 (V-)
- net VBAT: now also K1.4, K1.6, R7.3
- net at U1.6 (OUT-): now also R10.1
- net at R8.1: now also R14.2, U3.6 (-)
- net at R8.2: now also U3.7, U4.3 (+)
- net at U2.6 (OUT-): now also R14.1
- net at U1.7 (OUT+): now also R9.1
- net at U2.7 (OUT+): now also R13.1
- net VBAT_0.5%: no longer names the net of C6.1, R5.2, R6.1, U2.2 (IN)
- net VCAP_0.5%: no longer names the net of C5.1, R2.2, R3.1, U1.2 (IN)
- new net: R11.2, R9.2, U3.3 (+)
- new net: D3.1 (K), R17.1
- new net: R13.2, R15.2, U3.5 (+)
- new net: K1.3, K1.5, R7.1
- new net: D2.1 (K), R16.1
- new net: R10.2, R12.1, U3.2 (-)
- new net: R12.2, U3.1, U4.1 (-)
- new net CHARGE-EN: D1.1 (K), D3.2 (A), K1.2, Q1.3 (D), Q1.6 (D)
Other:
- moved on the sheet: R1, R2, R3, R6, R8
