File: Discharge/discharge.kicad_sch (KiCad schematic)
At the start: 4 parts, among them J1 HV_Conn_IN, J2 LV_Conn_IN

Commit message: Add files via upload
Parts:
- removed IMB06IGR1: S1, customFootprints:IMB03IGR, symbol Relay:G5Q-1
- added 12V1: K1, customFootprints:G9KB1ADC12, symbol Relay:G5Q-1
- added J1x1, J4: REL_COIL, molexMiniFitJr:MFJ_2X1, symbol Connector_Generic:Conn_01x02
- added J2x1, J3: REL_SW, customFootprints:APP_ASMPR45-1X2-RK, symbol Connector_Generic:Conn_01x02
Connections:
- net +12V: now also J4.1 (Pin_1)
- net GND: now also J4.2 (Pin_2)
- net INV +: now also R1.2
- net INV -: now also J3.2 (Pin_2); no longer R1.1
- new net: J3.1 (Pin_1), R1.1
- new net: 12V1.1, J1x1.1 (Pin_1)
- new net: 12V1.8, J1x1.2 (Pin_2)
- new net: 12V1.3, J2x1.1 (Pin_1)
- new net: 12V1.6, J2x1.2 (Pin_2)
Other:
- moved on the sheet: J1, J2, R1

Commit message: Test
Parts:
- J2: value LV_Conn_IN -> LVS_Conn_IN
