File: Discharge/discharge.kicad_sch (KiCad schematic)
At the start: 8 parts, among them J1 HV_Conn_IN, J1x1 REL_COIL, J2 LVS_Conn_IN, J2x1 REL_SW, J3 REL_SW, J4 REL_COIL

Commit message: .
Parts:
- J2: value LVS_Conn_IN -> LV_Conn_IN
Changed lines of the file:
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@@
 			)
 		)
-		(property "Value" "LVS_Conn_IN"
+		(property "Value" "LV_Conn_IN"
 			(at 107.95 92.7099 0)
 			(effects
